File: hardware/macropad/dongle.kicad_sch (KiCad schematic)
At the start: 20 parts, among them J3 Conn_01x04_Pin, J5 USB_A, SW14 SW_Push, U1 AP2112K-3.3, U4 STM32F103C8Tx, U5 NRF24L01_Breakout, Y2 8Mhz

Commit message: updated bat switch, added 10k resistors. fixed fps
Parts:
- added R13, R14: 10k, Resistor_SMD:R_0805_2012Metric, symbol Device:R
Connections:
- net GND_DGL: now also R13.2, R14.2; no longer U4.20 (PB2), U4.44 (BOOT0)
- new net BOOT0_DGL: R14.1, U4.44 (BOOT0)
- new net BOOT1_DGL: R13.1, U4.20 (PB2)
Changed lines of the file:
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@@
 	)
 	(junction
-		(at 182.88 57.15)
-		(diameter 0)
-		(color 0 0 0 0)
-	)
-	(junction
 		(at 53.34 60.96)
 		(diameter 0)
@@
 	)
 	(junction
+		(at 186.69 57.15)
+		(diameter 0)
+		(color 0 0 0 0)
+	)
+	(junction
 		(at 250.19 21.59)
 		(diameter 0)
@@
 	(wire
 		(pts
-			(xy 184.15 53.34) (xy 184.15 57.15)
+			(xy 191.77 48.26) (xy 191.77 49.53)
 		)
 		(stroke
@@
 	(wire
 		(pts
-			(xy 181.61 57.15) (xy 182.88 57.15)
+			(xy 181.61 57.15) (xy 186.69 57.15)
 		)
 		(stroke
@@
 	(wire
 		(pts
-			(xy 181.61 53.34) (xy 181.61 57.15)
+			(xy 181.61 48.26) (xy 181.61 49.53)
 		)
 		(stroke
@@
 	(wire
 		(pts
-			(xy 184.15 57.15) (xy 182.88 57.15)
-		)
-		(stroke
-			(width 0)
-			(type default)
-		)
-	)
-	(wire
-		(pts
 			(xy 157.48 58.42) (xy 143.51 58.42)
 		)
@@
 	(wire
 		(pts
+			(xy 186.69 57.15) (xy 191.77 57.15)
+		)
+		(stroke
+			(width 0)
+			(type default)
+		)
+	)
+	(wire
+		(pts
 			(xy 48.26 90.17) (xy 55.88 90.17)
 		)
@@
 	)
 	(label "BOOT0_DGL"
-		(at 184.15 53.34 0)
+		(at 191.77 48.26 0)
 		(effects
 			(font
@@
 	)
 	(label "BOOT1_DGL"
-		(at 181.61 53.34 180)
+		(at 181.61 48.26 180)
 		(effects
 			(font
@@
 	(symbol
 		(lib_id "power:GND")
-		(at 182.88 57.15 0)
+		(at 186.69 57.15 0)
 		(unit 1)
 		(exclude_from_sim no)
@@
 		(fields_autoplaced yes)
 		(property "Reference" "#PWR0104"
-			(at 182.88 63.5 0)
+			(at 186.69 63.5 0)
 			(effects
 				(font
@@
 		)
 		(property "Value" "GND_DGL"
-			(at 185.42 58.4199 0)
+			(at 189.23 58.4199 0)
 			(effects
 				(font
@@
 		)
 		(property "Footprint" ""
-			(at 182.88 57.15 0)
+			(at 186.69 57.15 0)
 			(effects
 				(font
@@
 		)
 		(property "Datasheet" ""
-			(at 182.88 57.15 0)
+			(at 186.69 57.15 0)
 			(effects
 				(font
@@
 		)
 		(property "Description" "Power symbol creates a global label with name \"GND\" , ground"
-			(at 182.88 57.15 0)
+			(at 186.69 57.15 0)
 			(effects
 				(font
@@
 	)
 	(symbol
+		(lib_id "Device:R")
+		(at 181.61 53.34 0)
+		(unit 1)
+		(exclude_from_sim no)
+		(in_bom yes)
+		(on_board yes)
+		(dnp no)
+		(fields_autoplaced yes)
+		(property "Reference" "R13"
+			(at 184.15 52.0699 0)
+			(effects
+				(font
+					(size 1.27 1.27)
+				)
+				(justify left)
+			)
+		)
+		(property "Value" "10k"
+			(at 184.15 54.6099 0)
+			(effects
+				(font
+					(size 1.27 1.27)
+				)
+				(justify left)
+			)
+		)
+		(property "Footprint" "Resistor_SMD:R_0805_2012Metric"
+			(at 179.832 53.34 90)
+			(effects
+				(font
+					(size 1.27 1.27)
+				)
+				(hide yes)
+			)
+		)
+		(property "Datasheet" "~"
+			(at 181.61 53.34 0)
+			(effects
+				(font
+					(size 1.27 1.27)
+				)
+				(hide yes)
+			)
+		)
+		(property "Description" "Resistor"
+			(at 181.61 53.34 0)
+			(effects
+				(font
+					(size 1.27 1.27)
+				)
+				(hide yes)
+			)
+		)
+		(pin "1"
+		)
+		(pin "2"
+		)
+		(instances
+			(project ""
+				(path "/228dc472-b306-4e5f-8dc5-2bf23eb4978d/667b6152-bd4f-4e65-809f-60ee5320cd3d"
+					(reference "R13")
+					(unit 1)
+				)
+			)
+		)
+	)
+	(symbol
 		(lib_id "Device:C")
 		(at 59.69 27.94 0)
@@
 					(unit 1)
 				)
+			)
+		)
+	)
+	(symbol
+		(lib_id "Device:R")
+		(at 191.77 53.34 0)
+		(unit 1)
+		(exclude_from_sim no)
+		(in_bom yes)
+		(on_board yes)
+		(dnp no)
+		(fields_autoplaced yes)
+		(property "Reference" "R14"
+			(at 194.31 52.0699 0)
+			(effects
+				(font
+					(size 1.27 1.27)
+				)
+				(justify left)
+			)
+		)
+		(property "Value" "10k"
+			(at 194.31 54.6099 0)
+			(effects
+				(font
+					(size 1.27 1.27)
+				)
+				(justify left)
+			)
+		)
+		(property "Footprint" "Resistor_SMD:R_0805_2012Metric"
+			(at 189.992 53.34 90)
+			(effects
+				(font
+					(size 1.27 1.27)
+				)
+				(hide yes)
+			)
+		)
+		(property "Datasheet" "~"
+			(at 191.77 53.34 0)
+			(effects
+				(font
+					(size 1.27 1.27)
+				)
+				(hide yes)
+			)
+		)
+		(property "Description" "Resistor"
+			(at 191.77 53.34 0)
+			(effects
+				(font
+					(size 1.27 1.27)
+				)
+				(hide yes)
+			)
+		)
+		(pin "1"
+		)
+		(pin "2"
+		)
+		(instances
+			(project "macropad"
+				(path "/228dc472-b306-4e5f-8dc5-2bf23eb4978d/667b6152-bd4f-4e65-809f-60ee5320cd3d"
+					(reference "R14")
+					(unit 1)
+				)

Commit message: updated lp2992
Parts:
- removed U1: AP2112K-3.3, symbol Regulator_Linear:AP2112K-3.3
- added C6: 10n, symbol Device:C
- added U1: LP2992IM5-3.3/NOPB, LP2992:DBV0005A_M, symbol LP2992:LP2992IM5-3.3_NOPB
- C13: renamed from C16; value 1u -> 2.2u; footprint Capacitor_SMD:C_0805_2012Metric -> (none)
- renumbered C7 to C1, C22 to C10, C15 to C12, C10 to C2, C12 to C3, C13 to C4, C14 to C5, C19 to C7, C20 to C8, C21 to C9, J5 to J1, J3 to J2, R3 to R1, R13 to R2, R14 to R3, SW14 to SW10, U4 to U2, U5 to U3, Y2 to Y1
Connections:
- net +3.3V_DGL: now also U1.5 (OUT)
- net GND_DGL: now also C6.2, U1.2 (GND)
- net VBUS_DGL: now also U1.1 (IN), U1.3 (ON_OFF_N)
- new net: C6.1, U1.4 (BYP)
Other:
- moved on the sheet: C13, C2

Commit message: added usb-c receptacle footprint
Parts:
- renumbered C11 to C10, C3 to C11, C4 to C12, C2 to C13, C5 to C14, C12 to C15, C6 to C16, C7 to C19, C8 to C20, C13 to C21, C9 to C22, C10 to C23, C1 to C7, J2 to J3, J1 to J5, R3 to R13, R1 to R14, R2 to R3, SW10 to SW12, U2 to U4, U3 to U5, Y1 to Y2

Commit message: updated symbols. changed power. erc fixxed halfway
Parts:
- C16, C21: footprint (none) -> Capacitor_SMD:C_0603_1608Metric
- U1: footprint LP2992:DBV0005A_M -> LP2992:DBV0005A_N
- renumbered R13 to R5, R14 to R6, SW12 to SW10

Commit message: added usba fp, updated pcb, 5v to vbus
Parts:
- J5: footprint (none) -> usbA:U-G-O4DD-W-1
Changed lines of the file:
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@@
 			)
 		)
-		(property "Footprint" ""
+		(property "Footprint" "usbA:U-G-O4DD-W-1"
 			(at 185.42 116.84 0)
 			(effects

Commit message: replaced buttons with pads
Parts:
- removed SW10: SW_Push, Button_Switch_SMD:SW_Push_1P1T_NO_E-Switch_TL3301NxxxxxG, symbol Switch:SW_Push
- added J10: Conn_01x02, Connector_Wire:SolderWire-0.5sqmm_1x02_P4.6mm_D0.9mm_OD2.1mm, symbol Connector_Generic:Conn_01x02
- renumbered J3 to J5, J5 to J9
Connections:
- net GND_DGL: now also J10.2 (Pin_2)
- net NRST_DGL: now also J10.1 (Pin_1)
Changed lines of the file:
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@@
 	(wire
 		(pts
+			(xy 181.61 81.28) (xy 185.42 81.28)
+		)
+		(stroke
+			(width 0)
+			(type default)
+		)
+	)
+	(wire
+		(pts
 			(xy 191.77 81.28) (xy 191.77 90.17)
 		)
@@
 	(wire
 		(pts
+			(xy 187.96 81.28) (xy 191.77 81.28)
+		)
+		(stroke
+			(width 0)
+			(type default)
+		)
+	)
+	(wire
+		(pts
 			(xy 58.42 177.8) (xy 58.42 179.07)
 		)
@@
 		(dnp no)
 		(fields_autoplaced yes)
-		(property "Reference" "#PWR0102"
+		(property "Reference" "#PWR042"
 			(at 33.02 67.31 0)
 			(effects
@@
 				)
 				(path "/228dc472-b306-4e5f-8dc5-2bf23eb4978d/667b6152-bd4f-4e65-809f-60ee5320cd3d"
-					(reference "#PWR0102")
+					(reference "#PWR042")
 					(unit 1)
 				)
@@
 		(dnp no)
 		(fields_autoplaced yes)
-		(property "Reference" "#PWR0105"
+		(property "Reference" "#PWR044"
 			(at 44.45 116.84 0)
 			(effects
@@
 				)
 				(path "/228dc472-b306-4e5f-8dc5-2bf23eb4978d/667b6152-bd4f-4e65-809f-60ee5320cd3d"
-					(reference "#PWR0105")
+					(reference "#PWR044")
 					(unit 1)
 				)
@@
 		(dnp no)
 		(fields_autoplaced yes)
-		(property "Reference" "#PWR0101"
+		(property "Reference" "#PWR041"
 			(at 33.02 57.15 0)
 			(effects
@@
 				)
 				(path "/228dc472-b306-4e5f-8dc5-2bf23eb4978d/667b6152-bd4f-4e65-809f-60ee5320cd3d"
-					(reference "#PWR0101")
+					(reference "#PWR041")
+					(unit 1)
+				)
+			)
+		)
+	)
+	(symbol
+		(lib_id "Connector_Generic:Conn_01x02")
+		(at 185.42 76.2 90)
+		(unit 1)
+		(exclude_from_sim no)
+		(in_bom yes)
+		(on_board yes)
+		(dnp no)
+		(fields_autoplaced yes)
+		(property "Reference" "J10"
+			(at 190.5 74.9299 90)
+			(effects
+				(font
+					(size 1.27 1.27)
+				)
+				(justify right)
+			)
+		)
+		(property "Value" "Conn_01x02"
+			(at 190.5 77.4699 90)
+			(effects
+				(font
+					(size 1.27 1.27)
+				)
+				(justify right)
+			)
+		)
+		(property "Footprint" "Connector_Wire:SolderWire-0.5sqmm_1x02_P4.6mm_D0.9mm_OD2.1mm"
+			(at 185.42 76.2 0)
+			(effects
+				(font
+					(size 1.27 1.27)
+				)
+				(hide yes)
+			)
+		)
+		(property "Datasheet" "~"
+			(at 185.42 76.2 0)
+			(effects
+				(font
+					(size 1.27 1.27)
+				)
+				(hide yes)
+			)
+		)
+		(property "Description" "Generic connector, single row, 01x02, script generated (kicad-library-utils/schlib/autogen/connector/)"
+			(at 185.42 76.2 0)
+			(effects
+				(font
+					(size 1.27 1.27)
+				)
+				(hide yes)
+			)
+		)
+		(pin "2"
+		)
+		(pin "1"
+		)
+		(instances
+			(project "dongle"
+				(path "/228dc472-b306-4e5f-8dc5-2bf23eb4978d"
+					(reference "J3")
+					(unit 1)
+				)
+				(path "/228dc472-b306-4e5f-8dc5-2bf23eb4978d/667b6152-bd4f-4e65-809f-60ee5320cd3d"
+					(reference "J10")
 					(unit 1)
 				)
@@
 		(dnp no)
 		(fields_autoplaced yes)
-		(property "Reference" "#PWR0112"
+		(property "Reference" "#PWR049"
 			(at 186.69 63.5 0)
 			(effects
@@
 				)
 				(path "/228dc472-b306-4e5f-8dc5-2bf23eb4978d/667b6152-bd4f-4e65-809f-60ee5320cd3d"
-					(reference "#PWR0112")
+					(reference "#PWR049")
 					(unit 1)
 				)
@@
 		(on_board yes)
 		(dnp no)
-		(property "Reference" "#PWR0113"
+		(property "Reference" "#PWR048"
 			(at 125.73 116.84 0)
 			(effects
@@
 				)
 				(path "/228dc472-b306-4e5f-8dc5-2bf23eb4978d/667b6152-bd4f-4e65-809f-60ee5320cd3d"
-					(reference "#PWR0113")
+					(reference "#PWR048")
 					(unit 1)
 				)
@@
 		(dnp no)
 		(fields_autoplaced yes)
-		(property "Reference" "J3"
+		(property "Reference" "J5"
 			(at 177.165 17.78 0)
 			(effects
@@
 				)
 				(path "/228dc472-b306-4e5f-8dc5-2bf23eb4978d/667b6152-bd4f-4e65-809f-60ee5320cd3d"
-					(reference "J3")
+					(reference "J5")
 					(unit 1)
 				)
@@
 		(dnp no)
 		(fields_autoplaced yes)
-		(property "Reference" "#FLG0102"
+		(property "Reference" "#FLG02"
 			(at 50.8 175.895 0)
 			(effects
@@
 				)
 				(path "/228dc472-b306-4e5f-8dc5-2bf23eb4978d/667b6152-bd4f-4e65-809f-60ee5320cd3d"
-					(reference "#FLG0102")
+					(reference "#FLG02")
 					(unit 1)
 				)
@@
 		(dnp no)
 		(fields_autoplaced yes)
-		(property "Reference" "#PWR0106"
+		(property "Reference" "#PWR046"
 			(at 114.3 181.61 0)
 			(effects
@@
 				)
 				(path "/228dc472-b306-4e5f-8dc5-2bf23eb4978d/667b6152-bd4f-4e65-809f-60ee5320cd3d"
-					(reference "#PWR0106")
+					(reference "#PWR046")
 					(unit 1)
 				)
@@
 	)
 	(symbol
-		(lib_id "Switch:SW_Push")
-		(at 186.69 81.28 0)
-		(unit 1)
-		(exclude_from_sim no)
-		(in_bom yes)
-		(on_board yes)
-		(dnp no)
-		(fields_autoplaced yes)
-		(property "Reference" "SW10"
-			(at 186.69 73.66 0)
-			(effects
-				(font
-					(size 1.27 1.27)
-				)
-			)
-		)
-		(property "Value" "SW_Push"
-			(at 186.69 76.2 0)
-			(effects
-				(font
-					(size 1.27 1.27)
-				)
-			)
-		)
-		(property "Footprint" "Button_Switch_SMD:SW_Push_1P1T_NO_E-Switch_TL3301NxxxxxG"
-			(at 186.69 76.2 0)
-			(effects
-				(font
-					(size 1.27 1.27)
-				)
-				(hide yes)
-			)
-		)
-		(property "Datasheet" "~"
-			(at 186.69 76.2 0)
-			(effects
-				(font
-					(size 1.27 1.27)
-				)
-				(hide yes)
-			)
-		)
-		(property "Description" "Push button switch, generic, two pins"
-			(at 186.69 81.28 0)
-			(effects
-				(font
-					(size 1.27 1.27)
-				)
-				(hide yes)
-			)
-		)
-		(pin "2"
-		)
-		(pin "1"
-		)
-		(instances
-			(project ""
-				(path "/228dc472-b306-4e5f-8dc5-2bf23eb4978d"
-					(reference "SW10")
-					(unit 1)
-				)
-				(path "/228dc472-b306-4e5f-8dc5-2bf23eb4978d/667b6152-bd4f-4e65-809f-60ee5320cd3d"
-					(reference "SW10")
-					(unit 1)
-				)
-			)
-		)
-	)
-	(symbol
 		(lib_id "Device:C")
 		(at 33.02 57.15 0)
@@
 		(dnp no)
 		(fields_autoplaced yes)
-		(property "Reference" "#PWR0103"
+		(property "Reference" "#PWR047"
 			(at 125.73 30.48 0)
 			(effects
@@
 				)
 				(path "/228dc472-b306-4e5f-8dc5-2bf23eb4978d/667b6152-bd4f-4e65-809f-60ee5320cd3d"
-					(reference "#PWR0103")
+					(reference "#PWR047")
 					(unit 1)
 				)
@@
 		(dnp no)
 		(fields_autoplaced yes)
-		(property "Reference" "#FLG0101"
+		(property "Reference" "#FLG08"
 			(at 76.2 191.135 0)
 			(effects
@@
 				)
 				(path "/228dc472-b306-4e5f-8dc5-2bf23eb4978d/667b6152-bd4f-4e65-809f-60ee5320cd3d"
-					(reference "#FLG0101")
+					(reference "#FLG08")
 					(unit 1)
 				)
@@
 		(dnp no)
 		(fields_autoplaced yes)
-		(property "Reference" "#PWR0117"
+		(property "Reference" "#PWR056"
 			(at 250.19 24.13 0)
 			(effects
@@
 				)
 				(path "/228dc472-b306-4e5f-8dc5-2bf23eb4978d/667b6152-bd4f-4e65-809f-60ee5320cd3d"
-					(reference "#PWR0117")
+					(reference "#PWR056")
 					(unit 1)
 				)
@@
 		(dnp no)
 		(fields_autoplaced yes)
-		(property "Reference" "#PWR0114"
+		(property "Reference" "#PWR052"
 			(at 191.77 36.83 0)
 			(effects
@@
 				)
 				(path "/228dc472-b306-4e5f-8dc5-2bf23eb4978d/667b6152-bd4f-4e65-809f-60ee5320cd3d"
-					(reference "#PWR0114")
+					(reference "#PWR052")
 					(unit 1)
 				)
@@
 		(dnp no)
 		(fields_autoplaced yes)
-		(property "Reference" "#PWR0115"
+		(property "Reference" "#PWR051"
 			(at 191.77 26.67 0)
 			(effects
@@
 				)
 				(path "/228dc472-b306-4e5f-8dc5-2bf23eb4978d/667b6152-bd4f-4e65-809f-60ee5320cd3d"
-					(reference "#PWR0115")
+					(reference "#PWR051")
 					(unit 1)
 				)
@@
 		(dnp no)
 		(fields_autoplaced yes)
-		(property "Reference" "J5"
+		(property "Reference" "J9"
 			(at 181.61 102.87 0)
 			(effects
@@
 				)
 				(path "/228dc472-b306-4e5f-8dc5-2bf23eb4978d/667b6152-bd4f-4e65-809f-60ee5320cd3d"
-					(reference "J5")
+					(reference "J9")
 					(unit 1)
 				)
@@
 		(on_board yes)
 		(dnp no)
-		(property "Reference" "#PWR0111"
+		(property "Reference" "#PWR050"
 			(at 189.23 132.08 0)
 			(effects
@@
 				)
 				(path "/228dc472-b306-4e5f-8dc5-2bf23eb4978d/667b6152-bd4f-4e65-809f-60ee5320cd3d"
-					(reference "#PWR0111")
+					(reference "#PWR050")
 					(unit 1)
 				)
@@
 		(dnp no)
 		(fields_autoplaced yes)
-		(property "Reference" "#PWR0116"
+		(property "Reference" "#PWR057"
 			(at 250.19 59.69 0)
 			(effects
@@
 				)
 				(path "/228dc472-b306-4e5f-8dc5-2bf23eb4978d/667b6152-bd4f-4e65-809f-60ee5320cd3d"
-					(reference "#PWR0116")
+					(reference "#PWR057")
 					(unit 1)
 				)
@@
 		(on_board yes)
 		(dnp no)
-		(property "Reference" "#PWR0107"
+		(property "Reference" "#PWR043"
 			(at 43.18 181.61 0)
 			(effects
@@
 				)
 				(path "/228dc472-b306-4e5f-8dc5-2bf23eb4978d/667b6152-bd4f-4e65-809f-60ee5320cd3d"
-					(reference "#PWR0107")
+					(reference "#PWR043")
 					(unit 1)
 				)
@@
 		(dnp no)
 		(fields_autoplaced yes)
-		(property "Reference" "#PWR0104"
+		(property "Reference" "#PWR045"
 			(at 62.23 195.58 0)
 			(effects
@@
 				)
 				(path "/228dc472-b306-4e5f-8dc5-2bf23eb4978d/667b6152-bd4f-4e65-809f-60ee5320cd3d"
-					(reference "#PWR0104")
+					(reference "#PWR045")
 					(unit 1)
 				)
@@
 		(dnp no)
 		(fields_autoplaced yes)
-		(property "Reference" "#PWR0110"
+		(property "Reference" "#PWR055"
 			(at 199.39 110.49 0)
 			(effects
@@
 				)
 				(path "/228dc472-b306-4e5f-8dc5-2bf23eb4978d/667b6152-bd4f-4e65-809f-60ee5320cd3d"
-					(reference "#PWR0110")
+					(reference "#PWR055")
 					(unit 1)
 				)
@@
 		(dnp no)
 		(fields_autoplaced yes)
-		(property "Reference" "#PWR0109"
+		(property "Reference" "#PWR053"
 			(at 191.77 96.52 0)
 			(effects
@@
 				)
 				(path "/228dc472-b306-4e5f-8dc5-2bf23eb4978d/667b6152-bd4f-4e65-809f-60ee5320cd3d"
-					(reference "#PWR0109")
+					(reference "#PWR053")
 					(unit 1)
 				)
@@
 		(on_board yes)
 		(dnp no)
-		(property "Reference" "#PWR0108"
+		(property "Reference" "#PWR054"
 			(at 191.77 114.3 0)
 			(effects
@@
 				)
 				(path "/228dc472-b306-4e5f-8dc5-2bf23eb4978d/667b6152-bd4f-4e65-809f-60ee5320cd3d"
-					(reference "#PWR0108")
+					(reference "#PWR054")
 					(unit 1)
 				)

Commit message: updated. comments in whatsapp
Connections:
- net USB_D+_DGL renamed USB_D_DGL+
- net USB_D-_DGL renamed USB_D_DGL-
Changed lines of the file:
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@@
+		)
+	)
+	(label "USB_D_DGL-"
+		(at 157.48 63.5 180)
+		(effects
+			(font
+				(size 1.27 1.27)
+			)
+			(justify right bottom)
 		)
 	)
@@
 		)
 	)
-	(label "USB_D+_DGL"
-		(at 157.48 66.04 180)
-		(effects
-			(font
-				(size 1.27 1.27)
-			)
-			(justify right bottom)
-		)
-	)
 	(label "BOOT0_DGL"
 		(at 191.77 48.26 0)
@@
 		)
 	)
-	(label "USB_D-_DGL"
-		(at 157.48 63.5 180)
+	(label "USB_D_DGL+"
+		(at 157.48 66.04 180)
 		(effects
 			(font
@@
 		)
 	)
-	(label "USB_D-_DGL"
+	(label "USB_D_DGL-"
 		(at 209.55 118.11 0)
 		(effects
@@
 		)
 	)
-	(label "USB_D+_DGL"
+	(label "USB_D_DGL+"
 		(at 209.55 115.57 0)
 		(effects

Commit message: updated schematic and drc
Parts:
- added R22: 1M, Resistor_SMD:R_0603_1608Metric, symbol Device:R
Connections:
- net HSE_IN_DGL: now also R22.1
- net HSE_OUT_DGL: now also R22.2
Changed lines of the file:
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@@
+	(wire
+		(pts
+			(xy 39.37 78.74) (xy 30.48 78.74)
+		)
+		(stroke
+			(width 0)
+			(type default)
+		)
+	)
 	(wire
 		(pts
@@
 	(wire
 		(pts
+			(xy 30.48 78.74) (xy 30.48 90.17)
+		)
+		(stroke
+			(width 0)
+			(type default)
+		)
+	)
+	(wire
+		(pts
 			(xy 157.48 58.42) (xy 143.51 58.42)
 		)
@@
 	(wire
 		(pts
+			(xy 55.88 78.74) (xy 55.88 90.17)
+		)
+		(stroke
+			(width 0)
+			(type default)
+		)
+	)
+	(wire
+		(pts
 			(xy 227.33 29.21) (xy 237.49 29.21)
 		)
@@
 		(pts
 			(xy 48.26 90.17) (xy 55.88 90.17)
+		)
+		(stroke
+			(width 0)
+			(type default)
+		)
+	)
+	(wire
+		(pts
+			(xy 46.99 78.74) (xy 55.88 78.74)
 		)
 		(stroke
@@
 					(unit 1)
 				)
+			)
+		)
+	)
+	(symbol
+		(lib_id "Device:R")
+		(at 43.18 78.74 90)
+		(unit 1)
+		(exclude_from_sim no)
+		(in_bom yes)
+		(on_board yes)
+		(dnp no)
+		(fields_autoplaced yes)
+		(property "Reference" "R22"
+			(at 43.18 72.39 90)
+			(effects
+				(font
+					(size 1.27 1.27)
+				)
+			)
+		)
+		(property "Value" "1M"
+			(at 43.18 74.93 90)
+			(effects
+				(font
+					(size 1.27 1.27)
+				)
+			)
+		)
+		(property "Footprint" "Resistor_SMD:R_0603_1608Metric"
+			(at 43.18 80.518 90)
+			(effects
+				(font
+					(size 1.27 1.27)
+				)
+				(hide yes)
+			)
+		)
+		(property "Datasheet" "~"
+			(at 43.18 78.74 0)
+			(effects
+				(font
+					(size 1.27 1.27)
+				)
+				(hide yes)
+			)
+		)
+		(property "Description" "Resistor"
+			(at 43.18 78.74 0)
+			(effects
+				(font
+					(size 1.27 1.27)
+				)
+				(hide yes)
+			)
+		)
+		(pin "1"
+		)
+		(pin "2"
+		)
+		(instances
+			(project "macropad"
+				(path "/228dc472-b306-4e5f-8dc5-2bf23eb4978d/667b6152-bd4f-4e65-809f-60ee5320cd3d"
+					(reference "R22")
+					(unit 1)
+				)
