File: hardware/macropad/dongle.kicad_sch (KiCad schematic)
At the start: 24 parts, among them J10 Conn_01x02, J5 Conn_01x04_Pin, J9 USB_A, U1 LP2992IM5-3.3/NOPB, U4 STM32F103C8Tx, U5 NRF24L01_Breakout, Y2 8Mhz

Commit message: Macropad layout kinda done
Parts:
- U5: footprint RF_Module:nRF24L01_Breakout -> nrf24l01:nRF24L01_Breakout
Changed lines of the file:
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@@
 			)
 		)
-		(property "Footprint" "RF_Module:nRF24L01_Breakout"
+		(property "Footprint" "nrf24l01:nRF24L01_Breakout"
 			(at 254 21.59 0)
 			(effects

Commit message: updated dongle
Parts:
- J10: footprint Connector_Wire:SolderWire-0.5sqmm_1x02_P4.6mm_D0.9mm_OD2.1mm -> Connector_Hirose:Hirose_DF13-02P-1.25DSA_1x02_P1.25mm_Vertical
Changed lines of the file:
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@@
 			)
 		)
-		(property "Footprint" "Connector_Wire:SolderWire-0.5sqmm_1x02_P4.6mm_D0.9mm_OD2.1mm"
+		(property "Footprint" "Connector_Hirose:Hirose_DF13-02P-1.25DSA_1x02_P1.25mm_Vertical"
 			(at 185.42 76.2 0)
 			(effects

Commit message: stitching done
Connections:
- net GND_DGL renamed GND
Changed lines of the file:
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@@
 		)
 		(instances
-			(project "dongle"
+			(project "macropad"
 				(path "/228dc472-b306-4e5f-8dc5-2bf23eb4978d"
 					(reference "U3")
@@
 		)
 		(instances
-			(project "dongle"
+			(project "macropad"
 				(path "/228dc472-b306-4e5f-8dc5-2bf23eb4978d"
 					(reference "C7")
@@
 			)
 		)
-		(property "Value" "GND_DGL"
-			(at 35.56 62.2299 0)
+		(property "Value" "GND"
+			(at 33.02 66.04 0)
 			(effects
 				(font
 					(size 1.27 1.27)
 				)
-				(justify left)
 			)
 		)
@@
 		)
 		(instances
-			(project "dongle"
+			(project "macropad"
 				(path "/228dc472-b306-4e5f-8dc5-2bf23eb4978d"
 					(reference "#PWR04")
@@
 		)
 		(instances
-			(project "dongle"
+			(project "macropad"
 				(path "/228dc472-b306-4e5f-8dc5-2bf23eb4978d"
 					(reference "C6")
@@
 			)
 		)
-		(property "Value" "GND_DGL"
-			(at 46.99 111.7599 0)
+		(property "Value" "GND"
+			(at 44.45 115.57 0)
 			(effects
 				(font
 					(size 1.27 1.27)
 				)
-				(justify left)
 			)
 		)
@@
 		)
 		(instances
-			(project "dongle"
+			(project "macropad"
 				(path "/228dc472-b306-4e5f-8dc5-2bf23eb4978d"
 					(reference "#PWR01")
@@
 		)
 		(instances
-			(project "dongle"
+			(project "macropad"
 				(path "/228dc472-b306-4e5f-8dc5-2bf23eb4978d"
 					(reference "#PWR03")
@@
 		)
 		(instances
-			(project "dongle"
+			(project "macropad"
 				(path "/228dc472-b306-4e5f-8dc5-2bf23eb4978d"
 					(reference "J3")
@@
 			)
 		)
-		(property "Value" "GND_DGL"
-			(at 189.23 58.4199 0)
+		(property "Value" "GND"
+			(at 186.69 62.23 0)
 			(effects
 				(font
 					(size 1.27 1.27)
 				)
-				(justify left)
 			)
 		)
@@
 		)
 		(instances
-			(project "dongle"
+			(project "macropad"
 				(path "/228dc472-b306-4e5f-8dc5-2bf23eb4978d"
 					(reference "#PWR018")
@@
 			)
 		)
-		(property "Value" "GND_DGL"
+		(property "Value" "GND"
 			(at 125.476 114.808 0)
 			(effects
@@
 		)
 		(instances
-			(project "dongle"
+			(project "macropad"
 				(path "/228dc472-b306-4e5f-8dc5-2bf23eb4978d"
 					(reference "#PWR08")
@@
 		)
 		(instances
-			(project ""
+			(project "macropad"
 				(path "/228dc472-b306-4e5f-8dc5-2bf23eb4978d"
 					(reference "C11")
@@
 		)
 		(instances
-			(project "dongle"
+			(project "macropad"
 				(path "/228dc472-b306-4e5f-8dc5-2bf23eb4978d"
 					(reference "C10")
@@
 		)
 		(instances
-			(project "dongle"
+			(project "macropad"
 				(path "/228dc472-b306-4e5f-8dc5-2bf23eb4978d"
 					(reference "J2")
@@
 		)
 		(instances
-			(project "dongle"
+			(project "macropad"
 				(path "/228dc472-b306-4e5f-8dc5-2bf23eb4978d"
 					(reference "R1")
@@
 		)
 		(instances
-			(project "dongle"
+			(project "macropad"
 				(path "/228dc472-b306-4e5f-8dc5-2bf23eb4978d"
 					(reference "C8")
@@
 		)
 		(instances
-			(project "dongle"
+			(project "macropad"
 				(path "/228dc472-b306-4e5f-8dc5-2bf23eb4978d"
 					(reference "#FLG01")
@@
 		)
 		(instances
-			(project ""
+			(project "macropad"
 				(path "/228dc472-b306-4e5f-8dc5-2bf23eb4978d"
 					(reference "C9")
@@
 		)
 		(instances
-			(project "dongle"
+			(project "macropad"
 				(path "/228dc472-b306-4e5f-8dc5-2bf23eb4978d"
 					(reference "#PWR06")
@@
 		)
 		(instances
-			(project "dongle"
+			(project "macropad"
 				(path "/228dc472-b306-4e5f-8dc5-2bf23eb4978d"
 					(reference "C4")
@@
 		)
 		(instances
-			(project "dongle"
+			(project "macropad"
 				(path "/228dc472-b306-4e5f-8dc5-2bf23eb4978d"
 					(reference "C3")
@@
 		)
 		(instances
-			(project "dongle"
+			(project "macropad"
 				(path "/228dc472-b306-4e5f-8dc5-2bf23eb4978d"
 					(reference "#PWR07")
@@
 		)
 		(instances
-			(project "dongle"
+			(project "macropad"
 				(path "/228dc472-b306-4e5f-8dc5-2bf23eb4978d"
 					(reference "#FLG02")
@@
 		)
 		(instances
-			(project "dongle"
+			(project "macropad"
 				(path "/228dc472-b306-4e5f-8dc5-2bf23eb4978d"
 					(reference "C1")
@@
 		)
 		(instances
-			(project "dongle"
+			(project "macropad"
 				(path "/228dc472-b306-4e5f-8dc5-2bf23eb4978d"
 					(reference "#PWR016")
@@
 			)
 		)
-		(property "Value" "GND_DGL"
-			(at 194.31 31.7499 0)
+		(property "Value" "GND"
+			(at 191.77 35.56 0)
 			(effects
 				(font
 					(size 1.27 1.27)
 				)
-				(justify left)
 			)
 		)
@@
 		)
 		(instances
-			(project "dongle"
+			(project "macropad"
 				(path "/228dc472-b306-4e5f-8dc5-2bf23eb4978d"
 					(reference "#PWR013")
@@
 		)
 		(instances
-			(project "dongle"
+			(project "macropad"
 				(path "/228dc472-b306-4e5f-8dc5-2bf23eb4978d"
 					(reference "R2")
@@
 		)
 		(instances
-			(project "dongle"
+			(project "macropad"
 				(path "/228dc472-b306-4e5f-8dc5-2bf23eb4978d"
 					(reference "C13")
@@
 		)
 		(instances
-			(project "dongle"
+			(project "macropad"
 				(path "/228dc472-b306-4e5f-8dc5-2bf23eb4978d"
 					(reference "R3")
@@
 		)
 		(instances
-			(project "dongle"
+			(project "macropad"
 				(path "/228dc472-b306-4e5f-8dc5-2bf23eb4978d"
 					(reference "#PWR012")
@@
 		)
 		(instances
-			(project ""
+			(project "macropad"
 				(path "/228dc472-b306-4e5f-8dc5-2bf23eb4978d"
 					(reference "U1")
@@
 		)
 		(instances
-			(project ""
+			(project "macropad"
 				(path "/228dc472-b306-4e5f-8dc5-2bf23eb4978d"
 					(reference "J1")
@@
 		)
 		(instances
-			(project "dongle"
+			(project "macropad"
 				(path "/228dc472-b306-4e5f-8dc5-2bf23eb4978d"
 					(reference "C12")
@@
 			)
 		)
-		(property "Value" "GND_DGL"
+		(property "Value" "GND"
 			(at 186.69 131.064 0)
 			(effects
@@
 		)
 		(instances
-			(project "dongle"
+			(project "macropad"
 				(path "/228dc472-b306-4e5f-8dc5-2bf23eb4978d"
 					(reference "#PWR010")
@@
 			)
 		)
-		(property "Value" "GND_DGL"
-			(at 252.73 54.6099 0)
+		(property "Value" "GND"
+			(at 250.19 58.42 0)
 			(effects
 				(font
 					(size 1.27 1.27)
 				)
-				(justify left)
 			)
 		)
@@
 		)
 		(instances
-			(project "dongle"
+			(project "macropad"
 				(path "/228dc472-b306-4e5f-8dc5-2bf23eb4978d"
 					(reference "#PWR017")
@@
 		)
 		(instances
-			(project "dongle"
+			(project "macropad"
 				(path "/228dc472-b306-4e5f-8dc5-2bf23eb4978d"
 					(reference "C5")
@@
 		)
 		(instances
-			(project ""
+			(project "macropad"
 				(path "/228dc472-b306-4e5f-8dc5-2bf23eb4978d"
 					(reference "Y1")
@@
 		)
 		(instances
-			(project "dongle"
+			(project "macropad"
 				(path "/228dc472-b306-4e5f-8dc5-2bf23eb4978d"
 					(reference "#PWR02")
@@
 			)
 		)
-		(property "Value" "GND_DGL"
-			(at 64.77 190.4999 0)
+		(property "Value" "GND"
+			(at 62.23 194.31 0)
 			(effects
 				(font
 					(size 1.27 1.27)
 				)
-				(justify left)
 			)
 		)
@@
 		)
 		(instances
-			(project "dongle"
+			(project "macropad"
 				(path "/228dc472-b306-4e5f-8dc5-2bf23eb4978d"
 					(reference "#PWR05")
@@
 		)
 		(instances
-			(project "dongle"
+			(project "macropad"
 				(path "/228dc472-b306-4e5f-8dc5-2bf23eb4978d"
 					(reference "#PWR015")
@@
 		)
 		(instances
-			(project "dongle"
+			(project "macropad"
 				(path "/228dc472-b306-4e5f-8dc5-2bf23eb4978d"
 					(reference "U2")
@@
 		)
 		(instances
-			(project "dongle"
+			(project "macropad"
 				(path "/228dc472-b306-4e5f-8dc5-2bf23eb4978d"
 					(reference "C2")
@@
 			)
 		)
-		(property "Value" "GND_DGL"
+		(property "Value" "GND"
 			(at 191.77 95.25 0)
 			(effects
@@
 		)
 		(instances
-			(project ""
+			(project "macropad"
 				(path "/228dc472-b306-4e5f-8dc5-2bf23eb4978d"
 					(reference "#PWR041")
@@
 		)
 		(instances
-			(project "dongle"
+			(project "macropad"
 				(path "/228dc472-b306-4e5f-8dc5-2bf23eb4978d"
 					(reference "#PWR011")

Commit message: fab outputs
Parts:
- J10, J5, J9: now not fitted
- R6: value 1.5K -> 1.5k

Commit message: proper fab outs
Parts:
- C13: MPN (none) -> UMK212B7105KGHT
- R22: MPN (none) -> CRCW06031M00FKEA
- R6: MPN (none) -> RT0603FRE071K5L
Changed lines of the file:
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@@
+			)
+		)
+		(property "MPN" "RT0603FRE071K5L"
+			(at 199.39 111.76 0)
+			(effects
+				(font
+					(size 1.27 1.27)
+				)
+				(hide yes)
 			)
 		)
@@
 			)
 		)
+		(property "MPN" "CRCW06031M00FKEA"
+			(at 43.18 78.74 90)
+			(effects
+				(font
+					(size 1.27 1.27)
+				)
+				(hide yes)
+			)
+		)
 		(pin "1"
 		)
@@
 			(at 46.99 181.61 0)
 			(effects
+				(font
+					(size 1.27 1.27)
+				)
+				(hide yes)
+			)
+		)
+		(property "MPN" "UMK212B7105KGHT"
+			(at 46.99 181.61 0)
+			(effects

Commit message: fixed technical queries
Parts:
- C10, C15: footprint Capacitor_SMD:C_0603_1608Metric -> Capacitor_SMD:C_0201_0603Metric
- U5: now not fitted
Changed lines of the file:
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@@
 		(in_bom yes)
 		(on_board yes)
-		(dnp no)
+		(dnp yes)
 		(fields_autoplaced yes)
 		(property "Reference" "U5"
@@
 			)
 		)
-		(property "Footprint" "Capacitor_SMD:C_0603_1608Metric"
+		(property "Footprint" "Capacitor_SMD:C_0201_0603Metric"
 			(at 31.4452 106.68 0)
 			(effects
@@
 			)
 		)
-		(property "Footprint" "Capacitor_SMD:C_0603_1608Metric"
+		(property "Footprint" "Capacitor_SMD:C_0201_0603Metric"
 			(at 56.8452 106.68 0)
 			(effects
