File: hardware/macropad/_autosave-macropad.kicad_pcb (KiCad board)
At the start: 2 copper layers, 158.4 x 77 mm, 93 parts, among them J1 SWD, J10 Conn_01x02, J2 USB_C_Receptacle_USB2.0_16P, J3 Conn_01x02, J4 display(4x1), J5 Conn_01x04_Pin, J6 Conn_01x03_Socket, J8 Conn_01x02, J9 USB_A, Q1 Q_PMOS, Q2 FS8205A, SW1 SW_Push, SW10 SW_SPDT, SW12 RotaryEncoder_Switch, SW13 RotaryEncoder_Switch, SW2 SW_Push, SW3 SW_Push, SW4 SW_Push, SW5 SW_Push, SW6 SW_Push, SW7 SW_Push, SW8 SW_Push, SW9 SW_Push, U1 LP2992IM5-3.3/NOPB, U2 STM32F103C8Tx, U3 NRF24L01_Breakout, U4 STM32F103C8Tx, U5 NRF24L01_Breakout, U6 TP4056-42-ESOP8, U7 DW01A, U8 RT8010AGQW, U9 LP2992IM5-3.3/NOPB, Y1 8Mhz C_L=12pF, Y2 8Mhz

Commit message: routing
Parts:
- moved C9 14.3 mm to (125.2, 59.7), turned to 180 degrees
- moved C1 12.3 mm to (128.3, 63.2), turned to 90 degrees
- moved J3 11.7 mm to (124.5, 61.6), turned to 0 degrees
- moved C8 11.4 mm to (128.2, 70.4), turned to -90 degrees
- moved R2 11.0 mm to (114.5, 69.1), turned to 90 degrees
- moved C4 10.7 mm to (115.7, 72.7), turned to 180 degrees
- moved C5 10.6 mm to (127.4, 73.4), turned to 0 degrees
- moved R11 10.3 mm to (119.2, 60.4), turned to 180 degrees
- moved C6 10.2 mm to (128.2, 66.5)
- moved C2 10.0 mm to (116.0, 62.5)
- moved R12 10.00 mm to (123.3, 74.3), turned to 0 degrees
- moved Y1 4.58 mm to (101.0, 74.3)
- moved R21 4.39 mm to (104.1, 74.0)
- moved C18 3.66 mm to (101.6, 77.2)
- moved C17 3.53 mm to (102.4, 71.4)
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