File: hardware/macropad/macropad.kicad_sch (KiCad schematic)
At the start: 39 parts, among them J1 SWD, J2 USB_C_Receptacle_USB2.0_16P, J3 Conn_01x02, J4 display(4x1), SW1 SW_Push, SW12 RotaryEncoder_Switch, SW13 RotaryEncoder_Switch, SW2 SW_Push, SW3 SW_Push, SW4 SW_Push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

Commit message: updated schematic and drc
Parts:
- added R21: 1M, Resistor_SMD:R_0603_1608Metric, symbol Device:R
- added R23: 10k, Resistor_SMD:R_0805_2012Metric, symbol Device:R
- added R24: 5.1k, Resistor_SMD:R_0603_1608Metric, symbol Device:R
Connections:
- net ENC2CLK_PA4: no longer SW13.B, U2.14 (PA4)
- net ENC2DT_PA3: no longer SW13.A, U2.13 (PA3)
- net ENC2SW_PA8: no longer SW13.S1, U2.29 (PA8)
- net GND: now also R23.2
- net HSE_IN: now also R21.1
- net HSE_OUT: now also R21.2
- net VBUS: now also R24.2
- net ENC2CLK_PA9: now reaches U2.30 (PA9)
- net ENC2CLK_PA9: now also SW13.B
- net ENC2SW_PA10: now reaches U2.31 (PA10)
- net ENC2SW_PA10: now also SW13.S1
- new net ENC2DT_PA8: SW13.A, U2.29 (PA8)
- new net VBUS_DET: R23.1, R24.1, U2.13 (PA3)
- no-connect marks 9 -> 8
Other:
- moved on the sheet: C1, C17, C18, C2, C3, C4, C5, C6, C8, C9, J1, J3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

Commit message: Macropad layout kinda done
Parts:
- J1: footprint Connector_PinHeader_2.54mm:PinHeader_1x04_P2.54mm_Horizontal -> Connector_PinHeader_2.54mm:PinHeader_1x04_P2.54mm_Vertical
- U3: footprint RF_Module:nRF24L01_Breakout -> nrf24l01:nRF24L01_Breakout
Connections:
- net ENC2CLK_PA4 is gone; now on net ENC2DT_PA8: R20.1
- net ENC2DT_PA3 is gone; now on net ENC2CLK_PA9: R19.1
- net ENC2SW_PA8 is gone; now on net ENC2SW_PA10: R18.1
Changed lines of the file:
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@@
 		)
 	)
-	(label "ENC2DT_PA3"
-		(at 364.49 222.25 90)
-		(effects
-			(font
-				(size 1.27 1.27)
-			)
-			(justify left bottom)
-		)
-	)
 	(label "ENC2DT_PA8"
 		(at 365.76 31.75 180)
@@
 		)
 	)
+	(label "ENC2SW_PA10"
+		(at 368.3 222.25 90)
+		(effects
+			(font
+				(size 1.27 1.27)
+			)
+			(justify left bottom)
+		)
+	)
 	(label "USB_D+"
 		(at 204.47 110.49 0)
@@
 		)
 	)
-	(label "ENC2SW_PA8"
-		(at 368.3 222.25 90)
-		(effects
-			(font
-				(size 1.27 1.27)
-			)
-			(justify left bottom)
-		)
-	)
 	(label "K2"
 		(at 143.51 118.11 180)
@@
 		)
 	)
-	(label "ENC2CLK_PA4"
-		(at 360.68 222.25 90)
-		(effects
-			(font
-				(size 1.27 1.27)
-			)
-			(justify left bottom)
-		)
-	)
 	(label "ENC1CLK_PA1"
 		(at 314.96 36.83 180)
@@
 		)
 	)
+	(label "ENC2DT_PA8"
+		(at 360.68 222.25 90)
+		(effects
+			(font
+				(size 1.27 1.27)
+			)
+			(justify left bottom)
+		)
+	)
 	(label "K7"
 		(at 143.51 138.43 180)
@@
 		)
 	)
+	(label "ENC2CLK_PA9"
+		(at 364.49 222.25 90)
+		(effects
+			(font
+				(size 1.27 1.27)
+			)
+			(justify left bottom)
+		)
+	)
 	(label "ENC1SW_PA2"
 		(at 179.07 85.09 0)
@@
 			)
 		)
-		(property "Footprint" "Connector_PinHeader_2.54mm:PinHeader_1x04_P2.54mm_Horizontal"
+		(property "Footprint" "Connector_PinHeader_2.54mm:PinHeader_1x04_P2.54mm_Vertical"
 			(at 270.51 146.05 0)
 			(effects
@@
 			)
 		)
-		(property "Footprint" "RF_Module:nRF24L01_Breakout"
+		(property "Footprint" "nrf24l01:nRF24L01_Breakout"
 			(at 269.24 77.47 0)
 			(effects

Commit message: routing
Parts:
- J3: footprint Connector_Wire:SolderWire-0.5sqmm_1x02_P4.6mm_D0.9mm_OD2.1mm -> Connector_Hirose:Hirose_DF13-02P-1.25DSA_1x02_P1.25mm_Vertical
Changed lines of the file:
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@@
 			)
 		)
-		(property "Footprint" "Connector_Wire:SolderWire-0.5sqmm_1x02_P4.6mm_D0.9mm_OD2.1mm"
+		(property "Footprint" "Connector_Hirose:Hirose_DF13-02P-1.25DSA_1x02_P1.25mm_Vertical"
 			(at 46.99 57.15 0)
 			(effects

Commit message: routing-macropad(67)
Connections:
- net ENC1CLK_PA1: now also U2.30 (PA9); no longer U2.11 (PA1)
- net ENC1DT_PA0: now also U2.29 (PA8); no longer U2.10 (PA0)
- net ENC1SW_PA2: now also U2.31 (PA10); no longer U2.12 (PA2)
- net ENC2CLK_PA9: now also U2.11 (PA1); no longer U2.30 (PA9)
- net ENC2DT_PA8: now also U2.10 (PA0); no longer U2.29 (PA8)
- net ENC2SW_PA10: now also U2.12 (PA2); no longer U2.31 (PA10)
Changed lines of the file:
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@@
 	)
 	(label "ENC1CLK_PA1"
-		(at 179.07 82.55 0)
+		(at 179.07 102.87 0)
 		(effects
 			(font
@@
 	)
 	(label "ENC2DT_PA8"
-		(at 179.07 100.33 0)
+		(at 179.07 80.01 0)
 		(effects
 			(font
@@
 	)
 	(label "ENC2SW_PA10"
-		(at 179.07 105.41 0)
+		(at 179.07 85.09 0)
 		(effects
 			(font
@@
 	)
 	(label "ENC1DT_PA0"
-		(at 179.07 80.01 0)
+		(at 179.07 100.33 0)
 		(effects
 			(font
@@
 	)
 	(label "ENC2CLK_PA9"
-		(at 179.07 102.87 0)
+		(at 179.07 82.55 0)
 		(effects
 			(font
@@
 	)
 	(label "ENC1SW_PA2"
-		(at 179.07 85.09 0)
-		(effects
-			(font
+		(at 179.07 105.41 0)
+		(effects
+			(font

Commit message: stitching done
Changed lines of the file:
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@@
 		)
 		(instances
-			(project ""
+			(project "macropad"
 				(path "/228dc472-b306-4e5f-8dc5-2bf23eb4978d"
 					(reference "R2")
@@
 		)
 		(instances
-			(project ""
+			(project "macropad"
 				(path "/228dc472-b306-4e5f-8dc5-2bf23eb4978d"
 					(reference "R11")
@@
 		)
 		(instances
-			(project ""
+			(project "macropad"
 				(path "/228dc472-b306-4e5f-8dc5-2bf23eb4978d"
 					(reference "#PWR015")
@@
 		(on_board yes)
 		(dnp no)
-		(fields_autoplaced yes)
 		(property "Reference" "J2"
 			(at 355.6 134.62 0)
@@
 		)
 		(property "Footprint" "usbc:TYPE-C-SMD_U263-163N-4GS1735"
-			(at 359.41 157.48 0)
+			(at 360.172 185.166 0)
 			(effects
 				(font
 					(size 1.27 1.27)
 				)
-				(hide yes)
 			)
 		)
@@
 		)
 		(instances
-			(project ""
+			(project "macropad"
 				(path "/228dc472-b306-4e5f-8dc5-2bf23eb4978d"
 					(reference "J2")
@@
 		)
 		(instances
-			(project ""
+			(project "macropad"
 				(path "/228dc472-b306-4e5f-8dc5-2bf23eb4978d"
 					(reference "C9")
@@
 		)
 		(instances
-			(project ""
+			(project "macropad"
 				(path "/228dc472-b306-4e5f-8dc5-2bf23eb4978d"
 					(reference "SW12")

Commit message: fab outputs
Parts:
- J1, J3, J4, SW1, SW12, SW13, SW2, SW3, SW4, SW5, SW6, SW7, SW8, SW9: now not fitted
Changed lines of the file:
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@@
 		(in_bom yes)
 		(on_board yes)
-		(dnp no)
+		(dnp yes)
 		(fields_autoplaced yes)
 		(property "Reference" "SW8"
@@
 		(in_bom yes)
 		(on_board yes)
-		(dnp no)
+		(dnp yes)
 		(fields_autoplaced yes)
 		(property "Reference" "SW2"
@@
 		(in_bom yes)
 		(on_board yes)
-		(dnp no)
+		(dnp yes)
 		(fields_autoplaced yes)
 		(property "Reference" "SW4"
@@
 		(in_bom yes)
 		(on_board yes)
-		(dnp no)
+		(dnp yes)
 		(fields_autoplaced yes)
 		(property "Reference" "J1"
@@
 		(in_bom yes)
 		(on_board yes)
-		(dnp no)
+		(dnp yes)
 		(fields_autoplaced yes)
 		(property "Reference" "SW6"
@@
 		(in_bom yes)
 		(on_board yes)
-		(dnp no)
+		(dnp yes)
 		(fields_autoplaced yes)
 		(property "Reference" "SW9"
@@
 		(in_bom yes)
 		(on_board yes)
-		(dnp no)
+		(dnp yes)
 		(fields_autoplaced yes)
 		(property "Reference" "SW3"
@@
 		(in_bom yes)
 		(on_board yes)
-		(dnp no)
+		(dnp yes)
 		(fields_autoplaced yes)
 		(property "Reference" "SW13"
@@
 		(in_bom yes)
 		(on_board yes)
-		(dnp no)
+		(dnp yes)
 		(fields_autoplaced yes)
 		(property "Reference" "SW1"
@@
 		(in_bom yes)
 		(on_board yes)
-		(dnp no)
+		(dnp yes)
 		(fields_autoplaced yes)
 		(property "Reference" "J4"
@@
 		(in_bom yes)
 		(on_board yes)
-		(dnp no)
+		(dnp yes)
 		(fields_autoplaced yes)
 		(property "Reference" "SW5"
@@
 		(in_bom yes)
 		(on_board yes)
-		(dnp no)
+		(dnp yes)
 		(property "Reference" "J3"
 			(at 52.07 55.8799 90)
@@
 		(in_bom yes)
 		(on_board yes)
-		(dnp no)
+		(dnp yes)
 		(fields_autoplaced yes)
 		(property "Reference" "SW7"
@@
 		(in_bom yes)
 		(on_board yes)
-		(dnp no)
+		(dnp yes)
 		(fields_autoplaced yes)
 		(property "Reference" "SW12"

Commit message: proper fab outs
Parts:
- C18: MPN (none) -> GCM0335C1H180FA16D
- J2: MPN (none) -> U263-163N-4WS1735-XKB-5A
- R13: MPN (none) -> RC0805JR-0710KL
- R15: MPN (none) -> RT0603FRE075K1L
- SW12: MPN (none) -> KY-040
- U2: MPN (none) -> STM32F103C8T6
Changed lines of the file:
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@@
 			)
 		)
-		(property "Description" "Resistor"
+		(property "Description" "RC0805JR-0710KL"
+			(at 379.73 226.06 0)
+			(effects
+				(font
+					(size 1.27 1.27)
+				)
+				(hide yes)
+			)
+		)
+		(property "MPN" "RC0805JR-0710KL"
 			(at 379.73 226.06 0)
 			(effects
@@
 			)
 		)
-		(property "Description" "Resistor"
+		(property "Description" "RC0805JR-0710KL"
 			(at 44.45 101.6 0)
 			(effects
@@
 			)
 		)
+		(property "MPN" "U263-163N-4WS1735-XKB-5A"
+			(at 355.6 157.48 0)
+			(effects
+				(font
+					(size 1.27 1.27)
+				)
+				(hide yes)
+			)
+		)
 		(pin "B9"
 		)
@@
 			)
 		)
-		(property "Description" "Resistor"
+		(property "Description" "RC0805JR-0710KL"
 			(at 53.34 101.6 0)
 			(effects
@@
 			)
 		)
-		(property "Description" "Resistor"
+		(property "Description" "RC0805JR-0710KL"
 			(at 368.3 226.06 0)
 			(effects
@@
 			)
 		)
-		(property "Description" "Resistor"
+		(property "Description" "RC0805JR-0710KL"
 			(at 375.92 226.06 0)
 			(effects
@@
 			)
 		)
+		(property "MPN" "RT0603FRE075K1L"
+			(at 387.35 153.67 0)
+			(effects
+				(font
+					(size 1.27 1.27)
+				)
+				(hide yes)
+			)
+		)
 		(pin "1"
 		)
@@
 			)
 		)
+		(property "MPN" "STM32F103C8T6"
+			(at 161.29 113.03 0)
+			(effects
+				(font
+					(size 1.27 1.27)
+				)
+				(hide yes)
+			)
+		)
 		(pin "32"
 		)
@@
 			)
 		)
+		(property "MPN" "GCM0335C1H180FA16D"
+			(at 64.77 154.94 0)
+			(effects
+				(font
+					(size 1.27 1.27)
+				)
+				(hide yes)
+			)
+		)
 		(pin "1"
 		)
@@
 			)
 		)
-		(property "Description" "Resistor"
+		(property "Description" "RC0805JR-0710KL"
 			(at 372.11 226.06 0)
 			(effects
@@
 			)
 		)
-		(property "Description" "Resistor"
+		(property "Description" "RC0805JR-0710KL"
 			(at 360.68 226.06 0)
 			(effects
@@
 			)
 		)
+		(property "MPN" "KY-040"
+			(at 322.58 34.29 0)
+			(effects
+				(font
+					(size 1.27 1.27)
+				)
+				(hide yes)
+			)
+		)
 		(pin "B"
 		)
@@
 			)
 		)
-		(property "Description" "Resistor"
+		(property "Description" "RC0805JR-0710KL"
 			(at 364.49 226.06 0)
 			(effects

Commit message: fixed technical queries
Parts:
- C17, C18: footprint Capacitor_SMD:C_0603_1608Metric -> Capacitor_SMD:C_0201_0603Metric
- U3: now not fitted
Changed lines of the file:
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@@
 			)
 		)
-		(property "Footprint" "Capacitor_SMD:C_0603_1608Metric"
+		(property "Footprint" "Capacitor_SMD:C_0201_0603Metric"
 			(at 40.3352 158.75 0)
 			(effects
@@
 		(in_bom yes)
 		(on_board yes)
-		(dnp no)
+		(dnp yes)
 		(fields_autoplaced yes)
 		(property "Reference" "U3"
@@
 			)
 		)
-		(property "Footprint" "Capacitor_SMD:C_0603_1608Metric"
+		(property "Footprint" "Capacitor_SMD:C_0201_0603Metric"
 			(at 65.7352 158.75 0)
 			(effects
